Commit message: add: ur5e r2f140 implementation; TODO: joint limited & workstation options for all, add gripper, etc. impl. for ur3e and ur10e

File: ur_e_description/grippers/robotiq_2f_140/urdf/robotiq_2f_140_macro.xacro (robot description, xacro)
@@ -2,5 +2,5 @@
 <robot name="robotiq_arg2f_140_model" xmlns:xacro="http://ros.org/wiki/xacro">
   <xacro:macro name="load_gripper" params="parent prefix">
-    <xacro:include filename="$(find kortex_description)/grippers/robotiq_2f_140/urdf/robotiq_arg2f_140_model_macro.xacro" />
+    <xacro:include filename="$(find ur_e_description)/grippers/robotiq_2f_140/urdf/robotiq_arg2f_140_model_macro.xacro" />
     <xacro:robotiq_arg2f_140 parent="${parent}" prefix="${prefix}"/>
   </xacro:macro>

File: ur_e_description/grippers/robotiq_2f_140/urdf/robotiq_2f_140_transmission_macro.xacro (robot description, xacro)
@@ -55,6 +55,7 @@
             <plugin name="gazebo_grasp_fix" filename="libgazebo_grasp_fix.so">
                 <arm>
-                    <arm_name>my_robotiq_gripper</arm_name>
-                    <palm_link>${prefix}bracelet_link</palm_link> <!-- Gazebo merges links connected by fixed joints, so here we would have put gripper_base_link but it is merged with Bracelet_Link internally -->
+                    <arm_name>ur5e</arm_name>
+                    <palm_link>${prefix}wrist_3_link</palm_link>
+                    <!-- Gazebo merges links connected by fixed joints, so you need to check the links in gazebo and choose one that is recognized after internal connections are made. We would want to choose the actual paml of the gripper but it is currently not an option -->
                     <gripper_link> ${prefix}left_inner_finger </gripper_link>
                     <gripper_link> ${prefix}right_inner_finger </gripper_link>

File: ur_e_description/grippers/robotiq_2f_140/urdf/robotiq_arg2f.xacro (robot description, xacro)
@@ -3,8 +3,9 @@
   <xacro:macro name="robotiq_arg2f_base_link" params="parent prefix">
     <!-- This joint was added by Kinova -->
+    <!-- The rotation on this joint has been edited to attach to the URe robots -->
     <joint name="${prefix}gripper_base_joint" type="fixed">
         <parent link="${parent}"/>
         <child link="${prefix}robotiq_arg2f_base_link"/>
-        <origin rpy="0.0 0.0 1.57" xyz="0.0 0.0 0.0"/>
+        <origin rpy="0.0 ${pi/2} 0.0" xyz="0.0 0.0 0.0"/>
     </joint>
     <link name="${prefix}robotiq_arg2f_base_link">
@@ -18,6 +19,6 @@
         <geometry>
           <!-- The DAE file doesn't show well in Gazebo so we're using the STL instead -->
-          <!-- <mesh filename="package://kortex_description/grippers/robotiq_2f_140/meshes/visual/robotiq_arg2f_140_base_link.dae" scale="0.001 0.001 0.001"/> -->
-          <mesh filename="package://kortex_description/grippers/robotiq_2f_140/meshes/collision/robotiq_arg2f_base_link.stl" />
+          <!-- <mesh filename="package://ur_e_description/grippers/robotiq_2f_140/meshes/visual/robotiq_arg2f_140_base_link.dae" scale="0.001 0.001 0.001"/> -->
+          <mesh filename="package://ur_e_description/grippers/robotiq_2f_140/meshes/collision/robotiq_arg2f_base_link.stl" />
         </geometry>
         <material name="">
@@ -28,5 +29,5 @@
         <origin xyz="0 0 0" rpy="0 0 0" />
         <geometry>
-          <mesh filename="package://kortex_description/grippers/robotiq_2f_140/meshes/collision/robotiq_arg2f_base_link.stl" />
+          <mesh filename="package://ur_e_description/grippers/robotiq_2f_140/meshes/collision/robotiq_arg2f_base_link.stl" />
         </geometry>
       </collision>

File: ur_e_description/grippers/robotiq_2f_140/urdf/robotiq_arg2f_140_model_macro.xacro (robot description, xacro)
@@ -17,5 +17,5 @@
         <origin xyz="0 0 0" rpy="0 0 0" />
         <geometry>
-          <mesh filename="package://kortex_description/grippers/robotiq_2f_140/meshes/visual/robotiq_arg2f_${stroke}_outer_knuckle.stl" />
+          <mesh filename="package://ur_e_description/grippers/robotiq_2f_140/meshes/visual/robotiq_arg2f_${stroke}_outer_knuckle.stl" />
         </geometry>
         <material name="">
@@ -26,5 +26,5 @@
         <origin xyz="0 0 0" rpy="0 0 0" />
         <geometry>
-          <mesh filename="package://kortex_description/grippers/robotiq_2f_140/meshes/collision/robotiq_arg2f_${stroke}_outer_knuckle.stl" />
+          <mesh filename="package://ur_e_description/grippers/robotiq_2f_140/meshes/collision/robotiq_arg2f_${stroke}_outer_knuckle.stl" />
         </geometry>
       </collision>
@@ -55,5 +55,5 @@
         <origin xyz="0 0 0" rpy="0 0 0" />
         <geometry>
-          <mesh filename="package://kortex_description/grippers/robotiq_2f_140/meshes/visual/robotiq_arg2f_${stroke}_outer_finger.stl" />
+          <mesh filename="package://ur_e_description/grippers/robotiq_2f_140/meshes/visual/robotiq_arg2f_${stroke}_outer_finger.stl" />
         </geometry>
         <material name="">
@@ -64,5 +64,5 @@
         <origin xyz="0 0 0" rpy="0 0 0" />
         <geometry>
-          <mesh filename="package://kortex_description/grippers/robotiq_2f_140/meshes/collision/robotiq_arg2f_${stroke}_outer_finger.stl" />
+          <mesh filename="package://ur_e_description/grippers/robotiq_2f_140/meshes/collision/robotiq_arg2f_${stroke}_outer_finger.stl" />
         </geometry>
       </collision>
@@ -88,5 +88,5 @@
         <origin xyz="0 0 0" rpy="0 0 0" />
         <geometry>
-          <mesh filename="package://kortex_description/grippers/robotiq_2f_140/meshes/visual/robotiq_arg2f_${stroke}_inner_knuckle.stl" />
+          <mesh filename="package://ur_e_description/grippers/robotiq_2f_140/meshes/visual/robotiq_arg2f_${stroke}_inner_knuckle.stl" />
         </geometry>
         <material name="">
@@ -97,5 +97,5 @@
         <origin xyz="0 0 0" rpy="0 0 0" />
         <geometry>
-          <mesh filename="package://kortex_description/grippers/robotiq_2f_140/meshes/collision/robotiq_arg2f_${stroke}_inner_knuckle.stl" />
+          <mesh filename="package://ur_e_description/grippers/robotiq_2f_140/meshes/collision/robotiq_arg2f_${stroke}_inner_knuckle.stl" />
         </geometry>
       </collision>
@@ -121,5 +121,5 @@
         <origin xyz="0 0 0" rpy="0 0 0" />
         <geometry>
-          <mesh filename="package://kortex_description/grippers/robotiq_2f_140/meshes/visual/robotiq_arg2f_${stroke}_inner_finger.stl" />
+          <mesh filename="package://ur_e_description/grippers/robotiq_2f_140/meshes/visual/robotiq_arg2f_${stroke}_inner_finger.stl" />
         </geometry>
         <material name="">
@@ -130,5 +130,5 @@
         <origin xyz="0 0 0" rpy="0 0 0" />
         <geometry>
-          <mesh filename="package://kortex_description/grippers/robotiq_2f_140/meshes/collision/robotiq_arg2f_${stroke}_inner_finger.stl" />
+          <mesh filename="package://ur_e_description/grippers/robotiq_2f_140/meshes/collision/robotiq_arg2f_${stroke}_inner_finger.stl" />
         </geometry>
       </collision>
@@ -197,5 +197,5 @@
     </joint>
   </xacro:macro>
-  <xacro:include filename="$(find kortex_description)/grippers/robotiq_2f_140/urdf/robotiq_arg2f.xacro" />
+  <xacro:include filename="$(find ur_e_description)/grippers/robotiq_2f_140/urdf/robotiq_arg2f.xacro" />
   <xacro:macro name="finger_joint" params="prefix">
     <joint name="${prefix}finger_joint" type="revolute">

File: ur_e_description/grippers/robotiq_2f_85/urdf/robotiq_arg2f.xacro (robot description, xacro)
@@ -3,4 +3,5 @@
   <xacro:macro name="robotiq_arg2f_base_link" params="parent prefix">
     <!-- This joint was added by Kinova -->
+    <!-- The rotation on this joint has been edited to attach to the URe robots -->
     <joint name="${prefix}gripper_base_joint" type="fixed">
         <parent link="${parent}"/>
@@ -28,5 +29,5 @@
         <origin xyz="0 0 0" rpy="0 0 0" />
         <geometry>
-           <mesh filename="package://ur_e_description/grippers/robotiq_2f_85/meshes/collision/robotiq_arg2f_base_link.stl" />
+          <mesh filename="package://ur_e_description/grippers/robotiq_2f_85/meshes/collision/robotiq_arg2f_base_link.stl" />
         </geometry>
       </collision>
