Commit message: edit: ur5e robot gripper/workstation configuration descriptions to actually spawn correct things; fix: launch errors due to typos pointing at wrong directory in some urdf macros; all current ur5e implementations functional

File: ur_e_description/urdf/ur3e_robot_robotiq_2f_140.urdf.xacro (robot description, xacro)
@@ -7,6 +7,6 @@
   <xacro:include filename="$(find ur_e_description)/urdf/ur3e.urdf.xacro" />
   <!-- robotiq_2f_140 -->
-  <xacro:include filename="$(find ur_e_description)/grippers/robotiq_2f_85/urdf/robotiq_2f_140_macro.xacro" />
-  <xacro:include filename="$(find ur_e_description)/grippers/robotiq_2f_85/urdf/robotiq_2f_140_transmission_macro.xacro" />
+  <xacro:include filename="$(find ur_e_description)/grippers/robotiq_2f_140/urdf/robotiq_2f_140_macro.xacro" />
+  <xacro:include filename="$(find ur_e_description)/grippers/robotiq_2f_140/urdf/robotiq_2f_140_transmission_macro.xacro" />
   <!-- arm -->
   <xacro:ur3e_robot prefix="" joint_limited="false"/>

File: ur_e_description/urdf/ur3e_robot_robotiq_2f_140_workstation.urdf.xacro (robot description, xacro)
@@ -9,6 +9,6 @@
   <xacro:include filename="$(find uml_hri_nerve_armada_workstation)/workstation_description/workstation_model.urdf.xacro" />
   <!-- robotiq_2f_140 -->
-  <xacro:include filename="$(find ur_e_description)/grippers/robotiq_2f_85/urdf/robotiq_2f_140_macro.xacro" />
-  <xacro:include filename="$(find ur_e_description)/grippers/robotiq_2f_85/urdf/robotiq_2f_140_transmission_macro.xacro" />
+  <xacro:include filename="$(find ur_e_description)/grippers/robotiq_2f_140/urdf/robotiq_2f_140_macro.xacro" />
+  <xacro:include filename="$(find ur_e_description)/grippers/robotiq_2f_140/urdf/robotiq_2f_140_transmission_macro.xacro" />
   <!-- arm -->
   <xacro:ur3e_robot prefix="" joint_limited="false"/>

File: ur_e_description/urdf/ur5e_joint_limited_robot_robotiq_2f_140.urdf.xacro (robot description, xacro)
@@ -1,14 +1,14 @@
 <?xml version="1.0"?>
 <robot xmlns:xacro="http://ros.org/wiki/xacro"
-       name="ur3e" >
+       name="ur5e" >
   <!-- common stuff -->
   <xacro:include filename="$(find ur_e_description)/urdf/common.gazebo.xacro" />
-  <!-- ur3e -->
-  <xacro:include filename="$(find ur_e_description)/urdf/ur3e.urdf.xacro" />
+  <!-- ur5e -->
+  <xacro:include filename="$(find ur_e_description)/urdf/ur5e.urdf.xacro" />
   <!-- robotiq_2f_140 -->
   <xacro:include filename="$(find ur_e_description)/grippers/robotiq_2f_140/urdf/robotiq_2f_140_macro.xacro" />
   <xacro:include filename="$(find ur_e_description)/grippers/robotiq_2f_140/urdf/robotiq_2f_140_transmission_macro.xacro" />
   <!-- arm -->
-  <xacro:ur3e_robot prefix="" joint_limited="true"
+  <xacro:ur5e_robot prefix="" joint_limited="true"
     shoulder_pan_lower_limit="${-pi}" shoulder_pan_upper_limit="${pi}"
     shoulder_lift_lower_limit="${-pi}" shoulder_lift_upper_limit="${pi}"

File: ur_e_description/urdf/ur5e_joint_limited_robot_robotiq_2f_140_workstation.urdf.xacro (robot description, xacro)
@@ -1,14 +1,16 @@
 <?xml version="1.0"?>
 <robot xmlns:xacro="http://ros.org/wiki/xacro"
-       name="ur3e" >
+       name="ur5e" >
   <!-- common stuff -->
   <xacro:include filename="$(find ur_e_description)/urdf/common.gazebo.xacro" />
-  <!-- ur3e -->
-  <xacro:include filename="$(find ur_e_description)/urdf/ur3e.urdf.xacro" />
+  <!-- ur5e -->
+  <xacro:include filename="$(find ur_e_description)/urdf/ur5e.urdf.xacro" />
+  <!-- ARMada workstation -->
+  <xacro:include filename="$(find uml_hri_nerve_armada_workstation)/workstation_description/workstation_model.urdf.xacro" />
   <!-- robotiq_2f_140 -->
   <xacro:include filename="$(find ur_e_description)/grippers/robotiq_2f_140/urdf/robotiq_2f_140_macro.xacro" />
   <xacro:include filename="$(find ur_e_description)/grippers/robotiq_2f_140/urdf/robotiq_2f_140_transmission_macro.xacro" />
   <!-- arm -->
-  <xacro:ur3e_robot prefix="" joint_limited="true"
+  <xacro:ur5e_robot prefix="" joint_limited="true"
     shoulder_pan_lower_limit="${-pi}" shoulder_pan_upper_limit="${pi}"
     shoulder_lift_lower_limit="${-pi}" shoulder_lift_upper_limit="${pi}"
@@ -21,9 +23,17 @@
   <xacro:load_gripper parent="ee_link"  prefix=""/>
   <xacro:load_gazebo_gripper_transmissions prefix=""/>
+  <!-- workstation -->
+  <xacro:workstation prefix="table_" namespace=""/>
   <link name="world" />
-  <joint name="world_joint" type="fixed">
+  <joint name="connect_world_and_table" type="fixed">
+    <child link="table_base_link" />
     <parent link="world" />
+    <origin xyz="0.0 0.0 0.41" rpy="0.0 0.0 0.0" />
+  </joint>
+  <!-- needs to be like kinova where root link is an argument -->
+  <joint name="connect_table_and_arm" type="fixed">
+    <parent link="table_mounting_plate_link" />
     <child link = "base_link" />
-    <origin xyz="0.0 0.0 0.0" rpy="0.0 0.0 0.0" />
+    <origin xyz="0.0 0.0 0.03625" rpy="0.0 0.0 ${pi/2}" />
   </joint>
 </robot>

File: ur_e_description/urdf/ur5e_joint_limited_robot_robotiq_2f_85.urdf.xacro (robot description, xacro)
@@ -1,14 +1,14 @@
 <?xml version="1.0"?>
 <robot xmlns:xacro="http://ros.org/wiki/xacro"
-       name="ur3e" >
+       name="ur5e" >
   <!-- common stuff -->
   <xacro:include filename="$(find ur_e_description)/urdf/common.gazebo.xacro" />
-  <!-- ur3e -->
-  <xacro:include filename="$(find ur_e_description)/urdf/ur3e.urdf.xacro" />
-  <!-- robotiq_2f_140 -->
-  <xacro:include filename="$(find ur_e_description)/grippers/robotiq_2f_140/urdf/robotiq_2f_140_macro.xacro" />
-  <xacro:include filename="$(find ur_e_description)/grippers/robotiq_2f_140/urdf/robotiq_2f_140_transmission_macro.xacro" />
+  <!-- ur5e -->
+  <xacro:include filename="$(find ur_e_description)/urdf/ur5e.urdf.xacro" />
+  <!-- robotiq_2f_85 -->
+  <xacro:include filename="$(find ur_e_description)/grippers/robotiq_2f_85/urdf/robotiq_2f_85_macro.xacro" />
+  <xacro:include filename="$(find ur_e_description)/grippers/robotiq_2f_85/urdf/robotiq_2f_85_transmission_macro.xacro" />
   <!-- arm -->
-  <xacro:ur3e_robot prefix="" joint_limited="true"
+  <xacro:ur5e_robot prefix="" joint_limited="true"
     shoulder_pan_lower_limit="${-pi}" shoulder_pan_upper_limit="${pi}"
     shoulder_lift_lower_limit="${-pi}" shoulder_lift_upper_limit="${pi}"

File: ur_e_description/urdf/ur5e_joint_limited_robot_robotiq_2f_85_workstation.urdf.xacro (robot description, xacro)
@@ -1,16 +1,16 @@
 <?xml version="1.0"?>
 <robot xmlns:xacro="http://ros.org/wiki/xacro"
-       name="ur3e" >
+       name="ur5e" >
   <!-- common stuff -->
   <xacro:include filename="$(find ur_e_description)/urdf/common.gazebo.xacro" />
-  <!-- ur3e -->
-  <xacro:include filename="$(find ur_e_description)/urdf/ur3e.urdf.xacro" />
+  <!-- ur5e -->
+  <xacro:include filename="$(find ur_e_description)/urdf/ur5e.urdf.xacro" />
   <!-- ARMada workstation -->
   <xacro:include filename="$(find uml_hri_nerve_armada_workstation)/workstation_description/workstation_model.urdf.xacro" />
-  <!-- robotiq_2f_140 -->
-  <xacro:include filename="$(find ur_e_description)/grippers/robotiq_2f_140/urdf/robotiq_2f_140_macro.xacro" />
-  <xacro:include filename="$(find ur_e_description)/grippers/robotiq_2f_140/urdf/robotiq_2f_140_transmission_macro.xacro" />
+  <!-- robotiq_2f_85 -->
+  <xacro:include filename="$(find ur_e_description)/grippers/robotiq_2f_85/urdf/robotiq_2f_85_macro.xacro" />
+  <xacro:include filename="$(find ur_e_description)/grippers/robotiq_2f_85/urdf/robotiq_2f_85_transmission_macro.xacro" />
   <!-- arm -->
-  <xacro:ur3e_robot prefix="" joint_limited="true"
+  <xacro:ur5e_robot prefix="" joint_limited="true"
     shoulder_pan_lower_limit="${-pi}" shoulder_pan_upper_limit="${pi}"
     shoulder_lift_lower_limit="${-pi}" shoulder_lift_upper_limit="${pi}"

File: ur_e_description/urdf/ur5e_robot_robotiq_2f_140.urdf.xacro (robot description, xacro)
@@ -6,5 +6,5 @@
   <!-- ur5e -->
   <xacro:include filename="$(find ur_e_description)/urdf/ur5e.urdf.xacro" />
-  <!-- robotiq_2f_85 -->
+  <!-- robotiq_2f_140 -->
   <xacro:include filename="$(find ur_e_description)/grippers/robotiq_2f_140/urdf/robotiq_2f_140_macro.xacro" />
   <xacro:include filename="$(find ur_e_description)/grippers/robotiq_2f_140/urdf/robotiq_2f_140_transmission_macro.xacro" />

File: ur_e_description/urdf/ur5e_robot_robotiq_2f_140_workstation.urdf.xacro (robot description, xacro)
@@ -6,7 +6,9 @@
   <!-- ur5e -->
   <xacro:include filename="$(find ur_e_description)/urdf/ur5e.urdf.xacro" />
-  <!-- robotiq_2f_85 -->
-  <xacro:include filename="$(find ur_e_description)/grippers/robotiq_2f_85/urdf/robotiq_2f_85_macro.xacro" />
-  <xacro:include filename="$(find ur_e_description)/grippers/robotiq_2f_85/urdf/robotiq_2f_85_transmission_macro.xacro" />
+  <!-- ARMada workstation -->
+  <xacro:include filename="$(find uml_hri_nerve_armada_workstation)/workstation_description/workstation_model.urdf.xacro" />
+  <!-- robotiq_2f_140 -->
+  <xacro:include filename="$(find ur_e_description)/grippers/robotiq_2f_140/urdf/robotiq_2f_140_macro.xacro" />
+  <xacro:include filename="$(find ur_e_description)/grippers/robotiq_2f_140/urdf/robotiq_2f_140_transmission_macro.xacro" />
   <!-- arm -->
   <xacro:ur5e_robot prefix="" joint_limited="false"/>
@@ -14,9 +16,17 @@
   <xacro:load_gripper parent="ee_link"  prefix=""/>
   <xacro:load_gazebo_gripper_transmissions prefix=""/>
+  <!-- workstation -->
+  <xacro:workstation prefix="table_" namespace=""/>
   <link name="world" />
-  <joint name="world_joint" type="fixed">
+  <joint name="connect_world_and_table" type="fixed">
+    <child link="table_base_link" />
     <parent link="world" />
+    <origin xyz="0.0 0.0 0.41" rpy="0.0 0.0 0.0" />
+  </joint>
+  <!-- needs to be like kinova where root link is an argument -->
+  <joint name="connect_table_and_arm" type="fixed">
+    <parent link="table_mounting_plate_link" />
     <child link = "base_link" />
-    <origin xyz="0.0 0.0 0.0" rpy="0.0 0.0 0.0" />
+    <origin xyz="0.0 0.0 0.03625" rpy="0.0 0.0 ${pi/2}" />
   </joint>
 </robot>

File: ur_e_description/urdf/ur5e_robot_robotiq_2f_85_workstation.urdf.xacro (robot description, xacro)
@@ -6,17 +6,27 @@
   <!-- ur5e -->
   <xacro:include filename="$(find ur_e_description)/urdf/ur5e.urdf.xacro" />
+  <!-- ARMada workstation -->
+  <xacro:include filename="$(find uml_hri_nerve_armada_workstation)/workstation_description/workstation_model.urdf.xacro" />
   <!-- robotiq_2f_85 -->
   <xacro:include filename="$(find ur_e_description)/grippers/robotiq_2f_85/urdf/robotiq_2f_85_macro.xacro" />
   <xacro:include filename="$(find ur_e_description)/grippers/robotiq_2f_85/urdf/robotiq_2f_85_transmission_macro.xacro" />
   <!-- arm -->
-  <xacro:ur5e_robot prefix="" joint_limited="false"/>
+  <xacro:ur5e_robot prefix="" joint_limited="false" />
   <!-- gripper -->
   <xacro:load_gripper parent="ee_link"  prefix=""/>
   <xacro:load_gazebo_gripper_transmissions prefix=""/>
+  <!-- workstation -->
+  <xacro:workstation prefix="table_" namespace=""/>
   <link name="world" />
-  <joint name="world_joint" type="fixed">
+  <joint name="connect_world_and_table" type="fixed">
+    <child link="table_base_link" />
     <parent link="world" />
+    <origin xyz="0.0 0.0 0.41" rpy="0.0 0.0 0.0" />
+  </joint>
+  <!-- needs to be like kinova where root link is an argument -->
+  <joint name="connect_table_and_arm" type="fixed">
+    <parent link="table_mounting_plate_link" />
     <child link = "base_link" />
-    <origin xyz="0.0 0.0 0.0" rpy="0.0 0.0 0.0" />
+    <origin xyz="0.0 0.0 0.03625" rpy="0.0 0.0 ${pi/2}" />
   </joint>
 </robot>
