Commit message: add: remaining current robot configuration descriptions for ur3,5,10e robots

File: ur_e_description/urdf/ur10e_joint_limited_robot_robotiq_2f_140.urdf.xacro (robot description, xacro)
@@ -10,5 +10,12 @@
   <xacro:include filename="$(find ur_e_description)/grippers/robotiq_2f_140/urdf/robotiq_2f_140_transmission_macro.xacro" />
   <!-- arm -->
-  <xacro:ur10e_robot prefix="" joint_limited="false"/>
+  <xacro:ur10e_robot prefix="" joint_limited="true"
+    shoulder_pan_lower_limit="${-pi}" shoulder_pan_upper_limit="${pi}"
+    shoulder_lift_lower_limit="${-pi}" shoulder_lift_upper_limit="${pi}"
+    elbow_joint_lower_limit="${-pi}" elbow_joint_upper_limit="${pi}"
+    wrist_1_lower_limit="${-pi}" wrist_1_upper_limit="${pi}"
+    wrist_2_lower_limit="${-pi}" wrist_2_upper_limit="${pi}"
+    wrist_3_lower_limit="${-pi}" wrist_3_upper_limit="${pi}"
+  />
   <!-- gripper -->
   <xacro:load_gripper parent="ee_link"  prefix=""/>

File: ur_e_description/urdf/ur10e_joint_limited_robot_robotiq_2f_140_workstation.urdf.xacro (robot description, xacro)
@@ -12,5 +12,12 @@
   <xacro:include filename="$(find ur_e_description)/grippers/robotiq_2f_140/urdf/robotiq_2f_140_transmission_macro.xacro" />
   <!-- arm -->
-  <xacro:ur10e_robot prefix="" joint_limited="false"/>
+  <xacro:ur10e_robot prefix="" joint_limited="true"
+    shoulder_pan_lower_limit="${-pi}" shoulder_pan_upper_limit="${pi}"
+    shoulder_lift_lower_limit="${-pi}" shoulder_lift_upper_limit="${pi}"
+    elbow_joint_lower_limit="${-pi}" elbow_joint_upper_limit="${pi}"
+    wrist_1_lower_limit="${-pi}" wrist_1_upper_limit="${pi}"
+    wrist_2_lower_limit="${-pi}" wrist_2_upper_limit="${pi}"
+    wrist_3_lower_limit="${-pi}" wrist_3_upper_limit="${pi}"
+  />
   <!-- gripper -->
   <xacro:load_gripper parent="ee_link"  prefix=""/>

File: ur_e_description/urdf/ur10e_joint_limited_robot_robotiq_2f_85.urdf.xacro (robot description, xacro)
@@ -10,5 +10,12 @@
   <xacro:include filename="$(find ur_e_description)/grippers/robotiq_2f_85/urdf/robotiq_2f_85_transmission_macro.xacro" />
   <!-- arm -->
-  <xacro:ur10e_robot prefix="" joint_limited="false"/>
+  <xacro:ur10e_robot prefix="" joint_limited="true"
+    shoulder_pan_lower_limit="${-pi}" shoulder_pan_upper_limit="${pi}"
+    shoulder_lift_lower_limit="${-pi}" shoulder_lift_upper_limit="${pi}"
+    elbow_joint_lower_limit="${-pi}" elbow_joint_upper_limit="${pi}"
+    wrist_1_lower_limit="${-pi}" wrist_1_upper_limit="${pi}"
+    wrist_2_lower_limit="${-pi}" wrist_2_upper_limit="${pi}"
+    wrist_3_lower_limit="${-pi}" wrist_3_upper_limit="${pi}"
+  />
   <!-- gripper -->
   <xacro:load_gripper parent="ee_link"  prefix=""/>

File: ur_e_description/urdf/ur10e_joint_limited_robot_robotiq_2f_85_workstation.urdf.xacro (robot description, xacro)
@@ -8,9 +8,16 @@
   <!-- ARMada workstation -->
   <xacro:include filename="$(find uml_hri_nerve_armada_workstation)/workstation_description/workstation_model.urdf.xacro" />
-  <!-- robotiq_2f_140 -->
-  <xacro:include filename="$(find ur_e_description)/grippers/robotiq_2f_140/urdf/robotiq_2f_140_macro.xacro" />
-  <xacro:include filename="$(find ur_e_description)/grippers/robotiq_2f_140/urdf/robotiq_2f_140_transmission_macro.xacro" />
+  <!-- robotiq_2f_85 -->
+  <xacro:include filename="$(find ur_e_description)/grippers/robotiq_2f_85/urdf/robotiq_2f_85_macro.xacro" />
+  <xacro:include filename="$(find ur_e_description)/grippers/robotiq_2f_85/urdf/robotiq_2f_85_transmission_macro.xacro" />
   <!-- arm -->
-  <xacro:ur10e_robot prefix="" joint_limited="false"/>
+  <xacro:ur10e_robot prefix="" joint_limited="true"
+    shoulder_pan_lower_limit="${-pi}" shoulder_pan_upper_limit="${pi}"
+    shoulder_lift_lower_limit="${-pi}" shoulder_lift_upper_limit="${pi}"
+    elbow_joint_lower_limit="${-pi}" elbow_joint_upper_limit="${pi}"
+    wrist_1_lower_limit="${-pi}" wrist_1_upper_limit="${pi}"
+    wrist_2_lower_limit="${-pi}" wrist_2_upper_limit="${pi}"
+    wrist_3_lower_limit="${-pi}" wrist_3_upper_limit="${pi}"
+  />
   <!-- gripper -->
   <xacro:load_gripper parent="ee_link"  prefix=""/>

File: ur_e_description/urdf/ur10e_robot_robotiq_2f_85_workstation.urdf.xacro (robot description, xacro)
@@ -1,22 +1,32 @@
 <?xml version="1.0"?>
 <robot xmlns:xacro="http://ros.org/wiki/xacro"
-       name="ur5e" >
+       name="ur10e" >
   <!-- common stuff -->
   <xacro:include filename="$(find ur_e_description)/urdf/common.gazebo.xacro" />
-  <!-- ur5e -->
-  <xacro:include filename="$(find ur_e_description)/urdf/ur5e.urdf.xacro" />
+  <!-- ur10e -->
+  <xacro:include filename="$(find ur_e_description)/urdf/ur10e.urdf.xacro" />
+  <!-- ARMada workstation -->
+  <xacro:include filename="$(find uml_hri_nerve_armada_workstation)/workstation_description/workstation_model.urdf.xacro" />
   <!-- robotiq_2f_85 -->
   <xacro:include filename="$(find ur_e_description)/grippers/robotiq_2f_85/urdf/robotiq_2f_85_macro.xacro" />
   <xacro:include filename="$(find ur_e_description)/grippers/robotiq_2f_85/urdf/robotiq_2f_85_transmission_macro.xacro" />
   <!-- arm -->
-  <xacro:ur5e_robot prefix="" joint_limited="false"/>
+  <xacro:ur10e_robot prefix="" joint_limited="false" />
   <!-- gripper -->
   <xacro:load_gripper parent="ee_link"  prefix=""/>
   <xacro:load_gazebo_gripper_transmissions prefix=""/>
+  <!-- workstation -->
+  <xacro:workstation prefix="table_" namespace=""/>
   <link name="world" />
-  <joint name="world_joint" type="fixed">
+  <joint name="connect_world_and_table" type="fixed">
+    <child link="table_base_link" />
     <parent link="world" />
+    <origin xyz="0.0 0.0 0.41" rpy="0.0 0.0 0.0" />
+  </joint>
+  <!-- needs to be like kinova where root link is an argument -->
+  <joint name="connect_table_and_arm" type="fixed">
+    <parent link="table_mounting_plate_link" />
     <child link = "base_link" />
-    <origin xyz="0.0 0.0 0.0" rpy="0.0 0.0 0.0" />
+    <origin xyz="0.0 0.0 0.03625" rpy="0.0 0.0 ${pi/2}" />
   </joint>
 </robot>
