Commit message: add: camera mount, millibar adapters models and macros, description files for adding hardware, update: gripper description to connect properly to moung structure, add: camera sim components to camera mount

File: ur_e_description/grippers/robotiq_2f_85/urdf/robotiq_arg2f.xacro (robot description, xacro)
@@ -7,5 +7,5 @@
         <parent link="${parent}"/>
         <child link="${prefix}robotiq_arg2f_base_link"/>
-        <origin rpy="0.0 ${pi/2} 0.0" xyz="0.0 0.0 0.0"/>
+        <origin rpy="0.0 0.0 ${pi/2}" xyz="0.0 0.0 0.0"/>
     </joint>
     <link name="${prefix}robotiq_arg2f_base_link">

File: ur_e_description/grippers/robotiq_2f_85/urdf/robotiq_arg2f_85_model_macro.xacro (robot description, xacro)
@@ -181,8 +181,7 @@
   <!-- Initialization of all joints and links -->
   <xacro:macro name="robotiq_arg2f_85" params="prefix parent">
-    <!-- Tool frame used by the arm -->
     <link name="${prefix}tool_frame"/>
     <joint name="${prefix}tool_frame_joint" type="fixed">
-        <origin xyz="0 0 0.120" rpy="${pi/2} 0 ${pi/2}" />
+        <origin xyz="0 0 0.120" rpy="0 0 0" />
         <parent link="${parent}" />
         <child link="${prefix}tool_frame" />
@@ -195,6 +194,4 @@
     <xacro:finger_joint prefix="${prefix}"/>
     <xacro:right_outer_knuckle_joint prefix="${prefix}"/>
-    <!-- Transmissions are loaded in the generic kortex xacro when simulation is enabled -->
-    <!-- <xacro:robotiq_arg2f_transmission prefix="${prefix}"/> -->
   </xacro:macro>
 </robot>

File: ur_e_description/urdf/ur5e.urdf.xacro (robot description, xacro)
@@ -320,5 +320,7 @@
       <parent link="${prefix}wrist_3_link" />
       <child link = "${prefix}ee_link" />
-      <origin xyz="0.0 ${wrist_3_length} 0.0" rpy="0.0 0.0 ${pi/2.0}" />
+      <!-- this is the original value -->
+      <!-- <origin xyz="0.0 ${wrist_3_length} 0.0" rpy="0.0 0.0 ${pi/2.0}" /> -->
+      <origin xyz="0.0 ${wrist_3_length} 0.0" rpy="-${pi/2.0} 0.0 0.0" />
     </joint>
     <link name="${prefix}ee_link">
